Commit message: adding lidar and camera

File: tracer/tracer_description/urdf/tracer_v1.xacro (robot description, xacro)
@@ -142,3 +142,96 @@
     <!-- Gazebo definitions  -->
     <xacro:include filename="$(find tracer_description)/urdf/tracer.gazebo" />
+    <!-- LiDAR Sensor -->
+<link name="lidar_link">
+  <visual>
+    <geometry>
+      <cylinder radius="0.04" length="0.05"/>
+    </geometry>
+    <origin xyz="0 0 0.1" rpy="0 0 0"/>
+  </visual>
+  <collision>
+    <geometry>
+      <cylinder radius="0.04" length="0.05"/>
+    </geometry>
+    <origin xyz="0 0 0.1" rpy="0 0 0"/>
+  </collision>
+  <inertial>
+    <mass value="0.1"/>
+    <origin xyz="0 0 0"/>
+    <inertia ixx="0.01" iyy="0.01" izz="0.01" ixy="0" ixz="0" iyz="0"/>
+  </inertial>
+</link>
+<joint name="lidar_joint" type="fixed">
+  <parent link="base_link"/>
+  <child link="lidar_link"/>
+  <origin xyz="0 0 0.35" rpy="0 0 0"/>
+</joint>
+<gazebo reference="lidar_link">
+  <sensor name="lidar_sensor" type="ray">
+    <update_rate>10</update_rate>
+    <ray>
+      <scan>
+        <horizontal>
+          <samples>360</samples>
+          <resolution>1</resolution>
+          <min_angle>-3.14</min_angle>
+          <max_angle>3.14</max_angle>
+        </horizontal>
+      </scan>
+      <range>
+        <min>0.1</min>
+        <max>10.0</max>
+      </range>
+      <noise>
+        <type>gaussian</type>
+        <mean>0.0</mean>
+        <stddev>0.01</stddev>
+      </noise>
+    </ray>
+    <plugin name="gazebo_ros_laser" filename="libgazebo_ros_ray_sensor.so">
+      <ros>
+        <namespace>/</namespace>
+      </ros>
+      <frame_name>lidar_link</frame_name>
+      <topic>/scan</topic>
+    </plugin>
+  </sensor>
+</gazebo>
+<!-- RGB Camera Sensor -->
+<link name="camera_link">
+  <visual>
+    <geometry>
+      <box size="0.04 0.04 0.04"/>
+    </geometry>
+    <origin xyz="0 0 0.1" rpy="0 0 0"/>
+  </visual>
+</link>
+<joint name="camera_joint" type="fixed">
+  <parent link="base_link"/>
+  <child link="camera_link"/>
+  <origin xyz="0.1 0 0.35" rpy="0 0 0"/>
+</joint>
+<gazebo reference="camera_link">
+  <sensor name="camera_sensor" type="camera">
+    <update_rate>30.0</update_rate>
+    <camera>
+      <horizontal_fov>1.39626</horizontal_fov>
+      <image>
+        <width>640</width>
+        <height>480</height>
+        <format>R8G8B8</format>
+      </image>
+      <clip>
+        <near>0.1</near>
+        <far>100</far>
+      </clip>
+    </camera>
+    <plugin name="gazebo_ros_camera" filename="libgazebo_ros_camera.so">
+      <camera_name>rgb_camera</camera_name>
+      <image_topic_name>/camera/image_raw</image_topic_name>
+      <camera_info_topic_name>/camera/camera_info</camera_info_topic_name>
+      <frame_name>camera_link</frame_name>
+    </plugin>
+  </sensor>
+</gazebo>
 </robot>

Commit message: working with lidar

File: tracer/tracer_description/urdf/tracer_v1.xacro (robot description, xacro)
@@ -170,23 +170,29 @@
   <sensor name="lidar_sensor" type="ray">
     <update_rate>10</update_rate>
-    <ray>
-      <scan>
-        <horizontal>
-          <samples>360</samples>
-          <resolution>1</resolution>
-          <min_angle>-3.14</min_angle>
-          <max_angle>3.14</max_angle>
-        </horizontal>
-      </scan>
-      <range>
-        <min>0.1</min>
-        <max>10.0</max>
-      </range>
-      <noise>
-        <type>gaussian</type>
-        <mean>0.0</mean>
-        <stddev>0.01</stddev>
-      </noise>
-    </ray>
+        <ray>
+          <scan>
+            <horizontal>
+              <samples>360</samples>
+              <resolution>1</resolution>
+              <min_angle>-3.14</min_angle>
+              <max_angle>3.14</max_angle>
+            </horizontal>
+            <vertical>
+              <samples>16</samples>   <!-- Adjust for vertical resolution -->
+              <resolution>1</resolution>
+              <min_angle>-0.3</min_angle>  <!-- Small downward tilt -->
+              <max_angle>0.3</max_angle>   <!-- Small upward tilt -->
+            </vertical>
+          </scan>
+          <range>
+            <min>0.1</min>
+            <max>10.0</max>
+          </range>
+          <noise>
+            <type>gaussian</type>
+            <mean>0.0</mean>
+            <stddev>0.01</stddev>
+          </noise>
+        </ray>
     <plugin name="gazebo_ros_laser" filename="libgazebo_ros_ray_sensor.so">
       <ros>
@@ -194,5 +200,5 @@
       </ros>
       <frame_name>lidar_link</frame_name>
-      <topic>/scan</topic>
+        <topic>/scan</topic>  <!-- This changes it -->
     </plugin>
   </sensor>
@@ -210,5 +216,5 @@
   <parent link="base_link"/>
   <child link="camera_link"/>
-  <origin xyz="0.1 0 0.35" rpy="0 0 0"/>
+  <origin xyz="0.1 0 0.35" rpy="-0.3 0"/>
 </joint>
 <gazebo reference="camera_link">
